File: PCB:Schematic/businessCard.kicad_pcb (KiCad board)
At the start: 2 copper layers, 85.6 x 54 mm, 48 parts, among them J1 Conn_01x07_Pin, J2 Conn_01x01_Pin, J3 Conn_01x01_Pin, Q1 MMBT3904, SW1 SW_Push, SW2 SW_Push, U1 XIAO-ESP32-C6, U2 BME280

Commit message: added updated pcb stuff
Routing:
- net +5V: track 241.4 -> 252.0 mm, vias 39 -> 38
- net SDA: track 27.7 -> 33.2 mm
- net Vibrator: track 41.0 -> 46.2 mm, vias 2 -> 3
- net Net-(D26-DOUT): track 5.42 -> 10.3 mm
- net Net-(D32-DOUT): track 5.46 -> 10.3 mm
- net Net-(D33-DOUT): track 5.45 -> 10.2 mm
- net Net-(D28-DOUT): track 5.44 -> 10.1 mm
- net Net-(D35-DOUT): track 5.45 -> 10.1 mm
- net Net-(D5-DOUT): track 5.48 -> 10.0 mm
- net Net-(D4-DOUT): track 5.49 -> 10.0 mm
- net Net-(D10-DOUT): track 5.49 -> 9.99 mm
- net Net-(D23-DOUT): track 5.44 -> 9.93 mm
- net Net-(D29-DOUT): track 5.41 -> 9.89 mm
- net Net-(D16-DOUT): track 5.53 -> 10.0 mm
- net Net-(D2-DOUT): track 5.56 -> 10.0 mm
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- added copper zone on B.Cu, net GND
- added copper zone on F.Cu, net GND
Other:
- board text added: "- explore tech - tinker - make cool stuff like this PCB - am a fast learner and adapter"
- board text removed: "- explore tech - tinker - make cool stuff like this PCB - am fast learner and adapter"
